Commit message: added controllers and teleoperate with keyboards

File: slamurai_description/urdf/slamurai.urdf.xacro (robot description, xacro)
@@ -1,11 +1,12 @@
 <?xml version="1.0"?>
-<!-- new line -->
 <robot name="slamurai" xmlns:xacro="http://ros.org/wiki/xacro">
- <link name="base_footprint"/>
- <link name="base_link">
-  <inertial>
-    <origin xyz="0.003143016747353246 0.20832048776027548 0.04035404903218986" rpy="0 0 0"/>
-    <mass value="2.175652670088412"/>
-    <inertia ixx="0.007647" iyy="0.012958" izz="0.020556" ixy="-0.0" iyz="0.0" ixz="-0.0"/>
+  <xacro:include filename="$(find slamurai_description)/urdf/slamurai_gazebo.xacro" />
+  <xacro:include filename="$(find slamurai_description)/urdf/slamurai_ros2_control.xacro" />
+<link name="base_footprint"/>
+<link name="base_link">
+  <inertial>
+    <origin xyz="-1.1773893992013494e-06 7.213238784553903e-17 0.037948219838041995" rpy="0 0 0"/>
+    <mass value="0.4493736051078449"/>
+    <inertia ixx="0.001778" iyy="0.002758" izz="0.004481" ixy="-0.0" iyz="-0.0" ixz="-0.0"/>
   </inertial>
   <visual>
@@ -26,54 +27,14 @@
     <parent link="base_footprint"/>
     <child link="base_link" />
-    <origin xyz="0 0 0.033" rpy="0 0 0"/>
+    <origin xyz="0 0 0" rpy="0 0 0"/>
   </joint>
-<link name="left1_motor1_1">
-  <inertial>
-    <origin xyz="-8.416856727366806e-06 0.03018842254028209 -1.376749971387925e-06" rpy="0 0 0"/>
-    <mass value="0.20727059427080408"/>
-    <inertia ixx="6.6e-05" iyy="1.5e-05" izz="6.6e-05" ixy="0.0" iyz="-0.0" ixz="0.0"/>
-  </inertial>
-  <visual>
-    <origin xyz="0.076857 -0.10832 -0.025412" rpy="0 0 0"/>
-    <geometry>
-      <mesh filename="file://$(find slamurai_description)/meshes/left1_motor1_1.stl" scale="0.001 0.001 0.001"/>
-    </geometry>
-    <material name="silver"/>
-  </visual>
-  <collision>
-    <origin xyz="0.076857 -0.10832 -0.025412" rpy="0 0 0"/>
-    <geometry>
-      <mesh filename="file://$(find slamurai_description)/meshes/left1_motor1_1.stl" scale="0.001 0.001 0.001"/>
-    </geometry>
-  </collision>
-</link>
-<link name="right_motor1_1">
-  <inertial>
-    <origin xyz="8.450351430322467e-06 -0.03018744701972803 -1.3767499708744468e-06" rpy="0 0 0"/>
-    <mass value="0.20727059427080408"/>
-    <inertia ixx="6.6e-05" iyy="1.5e-05" izz="6.6e-05" ixy="0.0" iyz="0.0" ixz="-0.0"/>
-  </inertial>
-  <visual>
-    <origin xyz="0.076857 -0.30832 -0.025412" rpy="0 0 0"/>
-    <geometry>
-      <mesh filename="file://$(find slamurai_description)/meshes/right_motor1_1.stl" scale="0.001 0.001 0.001"/>
-    </geometry>
-    <material name="silver"/>
-  </visual>
-  <collision>
-    <origin xyz="0.076857 -0.30832 -0.025412" rpy="0 0 0"/>
-    <geometry>
-      <mesh filename="file://$(find slamurai_description)/meshes/right_motor1_1.stl" scale="0.001 0.001 0.001"/>
-    </geometry>
-  </collision>
-</link>
 <link name="supportC_1">
   <inertial>
-    <origin xyz="1.6747352338253307e-08 4.877602759467692e-07 0.02749964776971598" rpy="0 0 0"/>
+    <origin xyz="-1.2351231148954867e-15 -1.1102230246251565e-16 0.027499999999997957" rpy="0 0 0"/>
     <mass value="0.03739064680839314"/>
     <inertia ixx="1e-05" iyy="1e-05" izz="1e-06" ixy="-0.0" iyz="0.0" ixz="0.0"/>
   </inertial>
   <visual>
-    <origin xyz="0.101857 -0.27832 -0.043412" rpy="0 0 0"/>
+    <origin xyz="0.105 -0.07 -0.045" rpy="0 0 0"/>
     <geometry>
       <mesh filename="file://$(find slamurai_description)/meshes/supportC_1.stl" scale="0.001 0.001 0.001"/>
@@ -82,5 +43,5 @@
   </visual>
   <collision>
-    <origin xyz="0.101857 -0.27832 -0.043412" rpy="0 0 0"/>
+    <origin xyz="0.105 -0.07 -0.045" rpy="0 0 0"/>
     <geometry>
       <mesh filename="file://$(find slamurai_description)/meshes/supportC_1.stl" scale="0.001 0.001 0.001"/>
@@ -90,10 +51,10 @@
 <link name="supportA_1">
   <inertial>
-    <origin xyz="1.674735296275376e-08 4.877602762243249e-07 0.027499647769715592" rpy="0 0 0"/>
+    <origin xyz="2.498001805406602e-16 8.326672684688674e-17 0.027499999999997166" rpy="0 0 0"/>
     <mass value="0.03739064680839313"/>
     <inertia ixx="1e-05" iyy="1e-05" izz="1e-06" ixy="-0.0" iyz="0.0" ixz="0.0"/>
   </inertial>
   <visual>
-    <origin xyz="0.101857 -0.13832 -0.043412" rpy="0 0 0"/>
+    <origin xyz="0.105 0.07 -0.045" rpy="0 0 0"/>
     <geometry>
       <mesh filename="file://$(find slamurai_description)/meshes/supportA_1.stl" scale="0.001 0.001 0.001"/>
@@ -102,5 +63,5 @@
   </visual>
   <collision>
-    <origin xyz="0.101857 -0.13832 -0.043412" rpy="0 0 0"/>
+    <origin xyz="0.105 0.07 -0.045" rpy="0 0 0"/>
     <geometry>
       <mesh filename="file://$(find slamurai_description)/meshes/supportA_1.stl" scale="0.001 0.001 0.001"/>
@@ -110,10 +71,10 @@
 <link name="supportD_1">
   <inertial>
-    <origin xyz="1.6747354072976783e-08 4.87760274975324e-07 0.027499647769715953" rpy="0 0 0"/>
+    <origin xyz="1.3739009929736312e-15 1.3877787807814457e-16 0.027499999999997554" rpy="0 0 0"/>
     <mass value="0.037390646808393165"/>
     <inertia ixx="1e-05" iyy="1e-05" izz="1e-06" ixy="-0.0" iyz="0.0" ixz="0.0"/>
   </inertial>
   <visual>
-    <origin xyz="-0.108143 -0.13832 -0.043412" rpy="0 0 0"/>
+    <origin xyz="-0.105 0.07 -0.045" rpy="0 0 0"/>
     <geometry>
       <mesh filename="file://$(find slamurai_description)/meshes/supportD_1.stl" scale="0.001 0.001 0.001"/>
@@ -122,5 +83,5 @@
   </visual>
   <collision>
-    <origin xyz="-0.108143 -0.13832 -0.043412" rpy="0 0 0"/>
+    <origin xyz="-0.105 0.07 -0.045" rpy="0 0 0"/>
     <geometry>
       <mesh filename="file://$(find slamurai_description)/meshes/supportD_1.stl" scale="0.001 0.001 0.001"/>
@@ -130,10 +91,10 @@
 <link name="supportB_1">
   <inertial>
-    <origin xyz="1.6747353559498634e-08 4.877602746700127e-07 0.02749964776971623" rpy="0 0 0"/>
+    <origin xyz="-1.3877787807814457e-17 -1.8041124150158794e-16 0.027499999999998193" rpy="0 0 0"/>
     <mass value="0.0373906468083932"/>
     <inertia ixx="1e-05" iyy="1e-05" izz="1e-06" ixy="-0.0" iyz="0.0" ixz="0.0"/>
   </inertial>
   <visual>
-    <origin xyz="-0.108143 -0.27832 -0.043412" rpy="0 0 0"/>
+    <origin xyz="-0.105 -0.07 -0.045" rpy="0 0 0"/>
     <geometry>
       <mesh filename="file://$(find slamurai_description)/meshes/supportB_1.stl" scale="0.001 0.001 0.001"/>
@@ -142,5 +103,5 @@
   </visual>
   <collision>
-    <origin xyz="-0.108143 -0.27832 -0.043412" rpy="0 0 0"/>
+    <origin xyz="-0.105 -0.07 -0.045" rpy="0 0 0"/>
     <geometry>
       <mesh filename="file://$(find slamurai_description)/meshes/supportB_1.stl" scale="0.001 0.001 0.001"/>
@@ -150,10 +111,10 @@
 <link name="top_link_1">
   <inertial>
-    <origin xyz="-0.10499998325264691 0.07000048776027559 0.002499647769714994" rpy="0 0 0"/>
-    <mass value="2.0891767604880593"/>
-    <inertia ixx="0.006804" iyy="0.01238" izz="0.019176" ixy="-0.0" iyz="0.0" ixz="0.0"/>
-  </inertial>
-  <visual>
-    <origin xyz="-0.108143 -0.13832 -0.098412" rpy="0 0 0"/>
+    <origin xyz="-0.10500000000000005 0.07000000000000002 0.002499999999996755" rpy="0 0 0"/>
+    <mass value="0.31617095432609105"/>
+    <inertia ixx="0.00103" iyy="0.001874" izz="0.002902" ixy="-0.0" iyz="0.0" ixz="0.0"/>
+  </inertial>
+  <visual>
+    <origin xyz="-0.105 0.07 -0.1" rpy="0 0 0"/>
     <geometry>
       <mesh filename="file://$(find slamurai_description)/meshes/top_link_1.stl" scale="0.001 0.001 0.001"/>
@@ -162,5 +123,5 @@
   </visual>
   <collision>
-    <origin xyz="-0.108143 -0.13832 -0.098412" rpy="0 0 0"/>
+    <origin xyz="-0.105 0.07 -0.1" rpy="0 0 0"/>
     <geometry>
       <mesh filename="file://$(find slamurai_description)/meshes/top_link_1.stl" scale="0.001 0.001 0.001"/>
@@ -168,132 +129,12 @@
   </collision>
 </link>
-<link name="left_motor2_1">
-  <inertial>
-    <origin xyz="-8.416856724008381e-06 0.030188422540280924 -1.3767499711381248e-06" rpy="0 0 0"/>
-    <mass value="0.20727059427080408"/>
-    <inertia ixx="6.6e-05" iyy="1.5e-05" izz="6.6e-05" ixy="0.0" iyz="-0.0" ixz="0.0"/>
-  </inertial>
-  <visual>
-    <origin xyz="-0.083143 -0.10832 -0.025412" rpy="0 0 0"/>
-    <geometry>
-      <mesh filename="file://$(find slamurai_description)/meshes/left_motor2_1.stl" scale="0.001 0.001 0.001"/>
-    </geometry>
-    <material name="silver"/>
-  </visual>
-  <collision>
-    <origin xyz="-0.083143 -0.10832 -0.025412" rpy="0 0 0"/>
-    <geometry>
-      <mesh filename="file://$(find slamurai_description)/meshes/left_motor2_1.stl" scale="0.001 0.001 0.001"/>
-    </geometry>
-  </collision>
-</link>
-<link name="right_motor2_1">
-  <inertial>
-    <origin xyz="-8.416856724466348e-06 -0.03018744701972903 6.72289406155463e-07" rpy="0 0 0"/>
-    <mass value="0.20727059427080408"/>
-    <inertia ixx="6.6e-05" iyy="1.5e-05" izz="6.6e-05" ixy="-0.0" iyz="-0.0" ixz="-0.0"/>
-  </inertial>
-  <visual>
-    <origin xyz="-0.083143 -0.30832 -0.025412" rpy="0 0 0"/>
-    <geometry>
-      <mesh filename="file://$(find slamurai_description)/meshes/right_motor2_1.stl" scale="0.001 0.001 0.001"/>
-    </geometry>
-    <material name="silver"/>
-  </visual>
-  <collision>
-    <origin xyz="-0.083143 -0.30832 -0.025412" rpy="0 0 0"/>
-    <geometry>
-      <mesh filename="file://$(find slamurai_description)/meshes/right_motor2_1.stl" scale="0.001 0.001 0.001"/>
-    </geometry>
-  </collision>
-</link>
-<link name="right_tyre2_1">
-  <inertial>
-    <origin xyz="1.6747331396671505e-08 0.012500487760274848 -3.522302838045166e-07" rpy="0 0 0"/>
-    <mass value="0.35728260237889004"/>
-    <inertia ixx="7.4e-05" iyy="0.000113" izz="7.4e-05" ixy="0.0" iyz="0.0" ixz="0.0"/>
-  </inertial>
-  <visual>
-    <origin xyz="-0.083143 -0.31832 -0.025412" rpy="0 0 0"/>
-    <geometry>
-      <mesh filename="file://$(find slamurai_description)/meshes/right_tyre2_1.stl" scale="0.001 0.001 0.001"/>
-    </geometry>
-    <material name="silver"/>
-  </visual>
-  <collision>
-    <origin xyz="-0.083143 -0.31832 -0.025412" rpy="0 0 0"/>
-    <geometry>
-      <mesh filename="file://$(find slamurai_description)/meshes/right_tyre2_1.stl" scale="0.001 0.001 0.001"/>
-    </geometry>
-  </collision>
-</link>
-<link name="right_tyre1_1">
-  <inertial>
-    <origin xyz="1.6747328565602793e-08 0.012500487760276957 -3.522302820836709e-07" rpy="0 0 0"/>
-    <mass value="0.3572826023788901"/>
-    <inertia ixx="7.4e-05" iyy="0.000113" izz="7.4e-05" ixy="0.0" iyz="0.0" ixz="0.0"/>
-  </inertial>
-  <visual>
-    <origin xyz="0.076857 -0.31832 -0.025412" rpy="0 0 0"/>
-    <geometry>
-      <mesh filename="file://$(find slamurai_description)/meshes/right_tyre1_1.stl" scale="0.001 0.001 0.001"/>
-    </geometry>
-    <material name="silver"/>
-  </visual>
-  <collision>
-    <origin xyz="0.076857 -0.31832 -0.025412" rpy="0 0 0"/>
-    <geometry>
-      <mesh filename="file://$(find slamurai_description)/meshes/right_tyre1_1.stl" scale="0.001 0.001 0.001"/>
-    </geometry>
-  </collision>
-</link>
-<link name="left_tyre1_1">
-  <inertial>
-    <origin xyz="1.6747329315003334e-08 -0.01249951223972294 -3.52230283124505e-07" rpy="0 0 0"/>
-    <mass value="0.3572826023788901"/>
-    <inertia ixx="7.4e-05" iyy="0.000113" izz="7.4e-05" ixy="0.0" iyz="0.0" ixz="0.0"/>
-  </inertial>
-  <visual>
-    <origin xyz="0.076857 -0.09832 -0.025412" rpy="0 0 0"/>
-    <geometry>
-      <mesh filename="file://$(find slamurai_description)/meshes/left_tyre1_1.stl" scale="0.001 0.001 0.001"/>
-    </geometry>
-    <material name="silver"/>
-  </visual>
-  <collision>
-    <origin xyz="0.076857 -0.09832 -0.025412" rpy="0 0 0"/>
-    <geometry>
-      <mesh filename="file://$(find slamurai_description)/meshes/left_tyre1_1.stl" scale="0.001 0.001 0.001"/>
-    </geometry>
-  </collision>
-</link>
-<link name="left_tyre2_1">
-  <inertial>
-    <origin xyz="1.6747330910948932e-08 -0.012499512239723787 -3.522302829163382e-07" rpy="0 0 0"/>
-    <mass value="0.3572826023788901"/>
-    <inertia ixx="7.4e-05" iyy="0.000113" izz="7.4e-05" ixy="0.0" iyz="0.0" ixz="0.0"/>
-  </inertial>
-  <visual>
-    <origin xyz="-0.083143 -0.09832 -0.025412" rpy="0 0 0"/>
-    <geometry>
-      <mesh filename="file://$(find slamurai_description)/meshes/left_tyre2_1.stl" scale="0.001 0.001 0.001"/>
-    </geometry>
-    <material name="silver"/>
-  </visual>
-  <collision>
-    <origin xyz="-0.083143 -0.09832 -0.025412" rpy="0 0 0"/>
-    <geometry>
-      <mesh filename="file://$(find slamurai_description)/meshes/left_tyre2_1.stl" scale="0.001 0.001 0.001"/>
-    </geometry>
-  </collision>
-</link>
 <link name="lidar_1">
   <inertial>
-    <origin xyz="0.03162534390052317 -0.13366928907724668 -0.00814920433767155" rpy="0 0 0"/>
+    <origin xyz="0.03476832715317002 0.07465122316247715 -0.009737852107389727" rpy="0 0 0"/>
     <mass value="1.338938753563966"/>
     <inertia ixx="0.000619" iyy="0.000967" izz="0.001105" ixy="-1e-06" iyz="-3e-06" ixz="0.000159"/>
   </inertial>
   <visual>
-    <origin xyz="0.098714 -0.346641 -0.146823" rpy="0 0 0"/>
+    <origin xyz="0.105 0.07 -0.15" rpy="0 0 0"/>
     <geometry>
       <mesh filename="file://$(find slamurai_description)/meshes/lidar_1.stl" scale="0.001 0.001 0.001"/>
@@ -302,5 +143,5 @@
   </visual>
   <collision>
-    <origin xyz="0.098714 -0.346641 -0.146823" rpy="0 0 0"/>
+    <origin xyz="0.105 0.07 -0.15" rpy="0 0 0"/>
     <geometry>
       <mesh filename="file://$(find slamurai_description)/meshes/lidar_1.stl" scale="0.001 0.001 0.001"/>
@@ -310,10 +151,10 @@
 <link name="buck_1">
   <inertial>
-    <origin xyz="0.011731735543703804 -0.24385518565506148 -0.03419369674872136" rpy="0 0 0"/>
+    <origin xyz="0.01487471879635087 -0.03553467341533718 -0.035782344518439646" rpy="0 0 0"/>
     <mass value="0.10059062602912178"/>
     <inertia ixx="3.2e-05" iyy="1.3e-05" izz="4.3e-05" ixy="0.0" iyz="-0.0" ixz="0.0"/>
   </inertial>
   <visual>
-    <origin xyz="-0.006286 -0.416641 -0.081823" rpy="0 0 0"/>
+    <origin xyz="0.0 0.0 -0.085" rpy="0 0 0"/>
     <geometry>
       <mesh filename="file://$(find slamurai_description)/meshes/buck_1.stl" scale="0.001 0.001 0.001"/>
@@ -322,5 +163,5 @@
   </visual>
   <collision>
-    <origin xyz="-0.006286 -0.416641 -0.081823" rpy="0 0 0"/>
+    <origin xyz="0.0 0.0 -0.085" rpy="0 0 0"/>
     <geometry>
       <mesh filename="file://$(find slamurai_description)/meshes/buck_1.stl" scale="0.001 0.001 0.001"/>
@@ -330,10 +171,10 @@
 <link name="cpu_1">
   <inertial>
-    <origin xyz="0.08988316113501907 -0.20987287386693915 -0.026296656222515966" rpy="0 0 0"/>
+    <origin xyz="0.093026144387666 -0.0015523616272141516 -0.027885303992234198" rpy="0 0 0"/>
     <mass value="0.5576753952846568"/>
     <inertia ixx="0.000337" iyy="0.000338" izz="0.000569" ixy="-1e-06" iyz="3e-06" ixz="4.1e-05"/>
   </inertial>
   <visual>
-    <origin xyz="-0.006286 -0.416641 -0.081823" rpy="0 0 0"/>
+    <origin xyz="0.0 0.0 -0.085" rpy="0 0 0"/>
     <geometry>
       <mesh filename="file://$(find slamurai_description)/meshes/cpu_1.stl" scale="0.001 0.001 0.001"/>
@@ -342,5 +183,5 @@
   </visual>
   <collision>
-    <origin xyz="-0.006286 -0.416641 -0.081823" rpy="0 0 0"/>
+    <origin xyz="0.0 0.0 -0.085" rpy="0 0 0"/>
     <geometry>
       <mesh filename="file://$(find slamurai_description)/meshes/cpu_1.stl" scale="0.001 0.001 0.001"/>
@@ -350,10 +191,10 @@
 <link name="motor_driver_1">
   <inertial>
-    <origin xyz="0.011019594541940285 -0.1636091685199691 -0.03094071532383927" rpy="0 0 0"/>
+    <origin xyz="0.01416257779458693 0.04471134371975541 -0.0325293630935574" rpy="0 0 0"/>
     <mass value="0.08494640552546982"/>
     <inertia ixx="1.4e-05" iyy="1.7e-05" izz="2.3e-05" ixy="0.0" iyz="-0.0" ixz="-3e-06"/>
   </inertial>
   <visual>
-    <origin xyz="-0.006286 -0.416641 -0.081823" rpy="0 0 0"/>
+    <origin xyz="0.0 0.0 -0.085" rpy="0 0 0"/>
     <geometry>
       <mesh filename="file://$(find slamurai_description)/meshes/motor_driver_1.stl" scale="0.001 0.001 0.001"/>
@@ -362,5 +203,5 @@
   </visual>
   <collision>
-    <origin xyz="-0.006286 -0.416641 -0.081823" rpy="0 0 0"/>
+    <origin xyz="0.0 0.0 -0.085" rpy="0 0 0"/>
     <geometry>
       <mesh filename="file://$(find slamurai_description)/meshes/motor_driver_1.stl" scale="0.001 0.001 0.001"/>
@@ -370,10 +211,10 @@
 <link name="mega_1">
   <inertial>
-    <origin xyz="-0.07038205492167375 -0.20893797511562137 -0.035610088672469134" rpy="0 0 0"/>
+    <origin xyz="-0.06723907166902694 -0.0006174628758972433 -0.03719873644218733" rpy="0 0 0"/>
     <mass value="0.11616477871692851"/>
     <inertia ixx="3.1e-05" iyy="0.00013" izz="0.000159" ixy="3e-06" iyz="0.0" ixz="-3e-06"/>
   </inertial>
   <visual>
-    <origin xyz="-0.006286 -0.416641 -0.081823" rpy="0 0 0"/>
+    <origin xyz="0.0 0.0 -0.085" rpy="0 0 0"/>
     <geometry>
       <mesh filename="file://$(find slamurai_description)/meshes/mega_1.stl" scale="0.001 0.001 0.001"/>
@@ -382,5 +223,5 @@
   </visual>
   <collision>
-    <origin xyz="-0.006286 -0.416641 -0.081823" rpy="0 0 0"/>
+    <origin xyz="0.0 0.0 -0.085" rpy="0 0 0"/>
     <geometry>
       <mesh filename="file://$(find slamurai_description)/meshes/mega_1.stl" scale="0.001 0.001 0.001"/>
@@ -388,31 +229,101 @@
   </collision>
 </link>
-<joint name="Rigid 8" type="fixed">
-  <origin xyz="-0.076857 0.10832 0.025412" rpy="0 0 0"/>
-  <parent link="base_link"/>
-  <child link="left1_motor1_1"/>
-</joint>
-<joint name="Rigid 9" type="fixed">
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
Commit message: harware codes updated

File: slamurai_description/urdf/slamurai.urdf.xacro (robot description, xacro)
@@ -1,4 +1,6 @@
 <?xml version="1.0"?>
 <robot name="slamurai" xmlns:xacro="http://ros.org/wiki/xacro">
+  <!-- Load Simulated or Real Hardware Interfaces -->
+  <xacro:arg name="is_sim" default="true"/>
   <xacro:include filename="$(find slamurai_description)/urdf/slamurai_gazebo.xacro" />
   <xacro:include filename="$(find slamurai_description)/urdf/slamurai_ros2_control.xacro" />

File: slamurai_description/urdf/slamurai_gazebo.xacro (robot description, xacro)
@@ -2,8 +2,4 @@
 <robot name="slamurai" xmlns:xacro="http://www.ros.org/wiki/xacro">
   <xacro:property name="body_color" value="Gazebo/Silver"/>
-  <!-- Material Definition -->
-  <material name="silver">
-    <color rgba="0.75 0.75 0.75 1.0"/>
-  </material>
   <!-- Move this one to ros2 control -->
   <transmission name="wheel_right_transmission">

File: slamurai_description/urdf/slamurai_ros2_control.xacro (robot description, xacro)
@@ -3,20 +3,29 @@
     <ros2_control name="RobotSystem" type="system">
         <!-- ros2_control Gazebo -->
-        <hardware>
-            <plugin>gazebo_ros2_control/GazeboSystem</plugin>
-        </hardware>
+        <xacro:if value="$(arg is_sim)">
+            <hardware>
+                <plugin>gazebo_ros2_control/GazeboSystem</plugin>
+            </hardware>
+        </xacro:if>
+        <!-- ros2_control Real Robot -->
+        <xacro:unless value="$(arg is_sim)">
+            <hardware>
+                <plugin>slamurai_firmware/slamuraiInterface</plugin>
+                <param name="port">/dev/arduino</param>
+            </hardware>
+        </xacro:unless>
         <!-- ros2_control Common Interfaces -->
-        <joint name="wheel_left_joint">
+        <joint name="wheel_right_joint">
             <command_interface name="velocity">
-              <param name="min">-10</param>
-              <param name="max">10</param>
+              <param name="min">-1</param>
+              <param name="max">1</param>
             </command_interface>
             <state_interface name="position" />
             <state_interface name="velocity" />
         </joint>
-        <joint name="wheel_right_joint">
+        <joint name="wheel_left_joint">
             <command_interface name="velocity">
-              <param name="min">-10</param>
-              <param name="max">10</param>
+              <param name="min">-1</param>
+              <param name="max">1</param>
             </command_interface>
             <state_interface name="position" />
